File: sensd/sensd.kicad_sch (KiCad schematic)
At the start: 60 parts, among them J1 Conn_01x05, J10 Conn_01x05, J11 Conn_01x05, J12 Conn_02x05_Top_Bottom, J13 RJ45, J14 DE9_Plug, J15 Conn_01x02, J2 Conn_01x05, J3 Conn_01x05, J4 Conn_01x05, J5 Conn_01x05, J6 Conn_01x05, J7 Conn_01x05, J8 Conn_01x05, J9 Conn_01x05, Q1 Q_NMOS_GSD, Q10 Q_NMOS_GSD, Q11 Q_NMOS_GSD, Q12 Q_NMOS_GSD, Q13 Q_NMOS_GSD, Q2 Q_NMOS_GSD, Q3 Q_NMOS_GSD, Q4 Q_NMOS_GSD, Q5 Q_NMOS_GSD, Q6 Q_NMOS_GSD, Q7 Q_NMOS_GSD, Q8 Q_NMOS_GSD, Q9 Q_NMOS_GSD, SW1 RotaryEncoder_Switch, U1 Teensy4.1, U2 MAX3232, U3 XL1509-5.0

Commit message: Nearly done with sch
Parts:
- added C5, C6: C_Polarized, Capacitor_SMD:CP_Elec_6.3x7.7, symbol Device:C_Polarized
- added D1: D, Diode_SMD:D_SMA, symbol Device:D
- added J16, J17: Conn_01x02, Connector_PinSocket_2.54mm:PinSocket_1x02_P2.54mm_Vertical, symbol Connector_Generic:Conn_01x02
- added J18: Conn_02x05_Top_Bottom, Connector_PinHeader_2.54mm:PinHeader_2x05_P2.54mm_Vertical, symbol Connector_Generic:Conn_02x05_Top_Bottom
- added L1: L, Inductor_SMD:L_7.3x7.3_H3.5, symbol Device:L
- added SW2, SW3, SW4, SW5: SW_Push, Button_Switch_Keyboard:SW_Cherry_MX_1.00u_PCB, symbol Switch:SW_Push
- R1: LCSC Part (none) -> C26000
Connections:
- net +12V: now also J15.2 (Pin_2), U3.1 (VIN), C5.1, J17.1 (Pin_1)
- net +3V3: now also R5.1
- net +5V: now also U3.3 (FB), C6.1, J16.1 (Pin_1), J18.1 (Pin_1), J18.6 (Pin_6), L1.2
- net GND: now also J15.1 (Pin_1), U3.4 (~{EN}), U3.5 (GND), U3.6 (GND), U3.7 (GND), U3.8 (GND), C5.2, C6.2, D1.2 (A), J18.2 (Pin_2), J18.7 (Pin_7), SW2.2, SW3.2, SW4.2, SW5.2
- net RX1: now also U1.2 (0_RX1_CRX2_CS1)
- net RX2: now also U1.9 (7_RX2_OUT1A)
- net RX3: now also U1.37 (15_A1_RX3_SPDIF_IN)
- net RX4: now also U1.20 (28_RX7)
- net RX5: now also U1.26 (34_RX8)
- net SCL1: now also U1.41 (19_A5_SCL)
- net SCL2: now also U1.38 (16_A2_RX4_SCL1)
- net SCL3: now also U1.16 (24_A10_TX6_SCL2)
- net SDA1: now also U1.40 (18_A4_SDA)
- net SDA2: now also U1.39 (17_A3_TX4_SDA1)
- net SDA3: now also U1.17 (25_A11_RX6_SDA2)
- net TX1: now also U1.3 (1_TX1_CTX2_MISO1)
- net TX2: now also U1.10 (8_TX2_IN1)
- net TX3: now also U1.36 (14_A0_TX3_SPDIF_OUT)
- net TX4: now also U1.21 (29_TX7)
- net TX5: now also U1.27 (35_TX8)
- net at Q13.3 (D): now also J17.2 (Pin_2)
- net at Q12.3 (D): now also J16.2 (Pin_2)
- net at U3.2 (OUT): now also D1.1 (K), L1.1
- new net CS: J18.8 (Pin_8)
- new net DC: J18.9 (Pin_9)
- new net MOSI: J18.3 (Pin_3)
- new net RES: J18.10 (Pin_10)
- new net SCK: J18.4 (Pin_4)
- new net SW2: SW2.1
- new net SW3: SW3.1
- new net SW4: SW4.1
- new net SW5: SW5.1
Other:
- moved on the sheet: J15

Commit message: board completed
Parts:
- removed J12: Conn_02x05_Top_Bottom, Connector_PinHeader_2.54mm:PinHeader_2x05_P2.54mm_Vertical, symbol Connector_Generic:Conn_02x05_Top_Bottom
- added D2: D, Diode_SMD:D_SMA, symbol Device:D
- added J12: Conn_01x02, Connector_AMASS:AMASS_XT30PW-F_1x02_P2.50mm_Horizontal, symbol Connector_Generic:Conn_01x02
- added JP10, JP11, JP12, JP13, JP15, JP16, JP17, JP18, JP19, JP2, JP20, JP21, JP22, JP23, JP27, JP28, JP29, JP3, JP30, JP31, JP32, JP33, JP34, JP35, JP36, JP38, JP39, JP4, JP40, JP41, JP42, JP43, JP44, JP45, JP5, JP6, JP7, JP8, JP9: SolderJumper_2_Open, Jumper:SolderJumper-2_P1.3mm_Open_TrianglePad1.0x1.5mm, symbol Jumper:SolderJumper_2_Open
- added Q14: Q_NMOS_GSD, Package_TO_SOT_SMD:SOT-23, symbol Device:Q_NMOS_GSD
- C1, C2, C3, C4: value C -> 100nF; LCSC Part (none) -> C1591
- C5, C6: value C_Polarized -> 220uF; LCSC Part (none) -> C2827940
- D1: LCSC Part (none) -> C85098
- L1: value L -> 33uH; LCSC Part (none) -> C3002653
- Q1, Q10, Q11, Q12, Q13, Q2, Q3, Q4, Q5, Q6, Q7, Q8, Q9: LCSC Part (none) -> C414015
- R10, R11, R12, R13, R14, R15, R16, R17, R18, R19, R2, R22, R23, R3, R4, R5, R6, R7, R8, R9: LCSC Part (none) -> C26000
- R20, R21: value R -> 0
- U2: LCSC Part (none) -> C45843
- U3: LCSC Part (none) -> C2902368
Connections:
- net +12V: now also J12.2 (Pin_2)
- net +5V: now also D2.1 (K)
- net A: now also JP38.2 (B)
- net B: now also JP39.2 (B)
- net CS: now also JP42.2 (B)
- net DC: now also JP22.1 (A)
- net FAN1: now also JP12.1 (A)
- net FAN2: now also JP11.1 (A)
- net FAN3: now also JP8.1 (A)
- net FAN4: now also JP28.2 (B)
- net FAN5: now also JP27.2 (B)
- net GND: now also BT1.2 (-), U1.52 (GND), Q14.2 (S)
- net HEATER: now also JP17.1 (A), Q14.1 (G)
- net MOSI: now also JP13.1 (A)
- net RES: now also JP21.1 (A)
- net RX1: now also JP2.1 (A); no longer U1.2 (0_RX1_CRX2_CS1)
- net RX2: now also JP9.1 (A); no longer U1.9 (7_RX2_OUT1A)
- net RX3: now also JP34.2 (B); no longer U1.37 (15_A1_RX3_SPDIF_IN)
- net RX4: now also JP19.1 (A); no longer U1.20 (28_RX7)
- net RX5: now also JP44.2 (B); no longer U1.26 (34_RX8)
- net SCK: now also JP36.2 (B)
- net SCL1: now also JP30.2 (B); no longer U1.41 (19_A5_SCL)
- net SCL2: now also JP33.2 (B); no longer U1.38 (16_A2_RX4_SCL1)
- net SCL3: now also JP15.1 (A); no longer U1.16 (24_A10_TX6_SCL2)
- net SDA1: now also JP31.2 (B); no longer U1.40 (18_A4_SDA)
- net SDA2: now also JP32.2 (B); no longer U1.39 (17_A3_TX4_SDA1)
- net SDA3: now also JP16.1 (A); no longer U1.17 (25_A11_RX6_SDA2)
- net SERVO1: now also JP4.1 (A)
- net SERVO2: now also JP5.1 (A)
- net SERVO3: now also JP6.1 (A)
- net SERVO4: now also JP7.1 (A)
- net SW1: now also JP40.2 (B)
- net SW2: now also JP41.2 (B)
- net SW3: now also JP29.2 (B)
- net SW4: now also JP23.1 (A)
- net SW5: now also JP45.2 (B)
- net TX1: now also JP3.1 (A); no longer U1.3 (1_TX1_CTX2_MISO1)
- net TX2: now also JP10.1 (A); no longer U1.10 (8_TX2_IN1)
- net TX3: now also JP35.2 (B); no longer U1.36 (14_A0_TX3_SPDIF_OUT)
- net TX4: now also JP20.1 (A); no longer U1.21 (29_TX7)
- net TX5: now also JP43.2 (B); no longer U1.27 (35_TX8)
- net WATER: now also JP18.1 (A)
- net at Q10.3 (D), Q11.3 (D), Q9.3 (D): now also J12.1 (Pin_1), Q14.3 (D)
- net at J16.2 (Pin_2), Q12.3 (D): now also D2.2 (A)
- net at U1.11 (9_OUT1C): now also JP11.2 (B)
- net at U1.12 (10_CS_MQSR): now also JP12.2 (B)
- net at U1.13 (11_MOSI_CTX1): now also JP13.2 (B)
- net at U1.18 (26_A12_MOSI1): now also JP17.2 (B)
- net at U1.19 (27_A13_SCK1): now also JP18.2 (B)
- net at U1.22 (30_CRX3): now also JP21.2 (B)
- net at U1.23 (31_CTX3): now also JP22.2 (B)
- net at U1.24 (32_OUT1B): now also JP23.2 (B)
- net at U1.25 (33_MCLK2): now also JP45.1 (A)
- net at U1.29 (37_CS): now also JP42.1 (A)
- net at U1.30 (38_CS1_IN1): now also JP41.1 (A)
- net at U1.31 (39_MISO1_OUT1A): now also JP40.1 (A)
- net at U1.32 (40_A16): now also JP39.1 (A)
- net at U1.33 (41_A17): now also JP38.1 (A)
- net at U1.35 (13_SCK_LED): now also JP36.1 (A)
- net at U1.4 (2_OUT2): now also JP4.2 (B)
- net at U1.42 (20_A6_TX5_LRCLK1): now also JP29.1 (A)
- net at U1.44 (22_A8_CTX1): now also JP28.1 (A)
- net at U1.45 (23_A9_CRX1_MCLK1): now also JP27.1 (A)
- net at U1.5 (3_LRCLK2): now also JP5.2 (B)
- net at U1.6 (4_BCLK2): now also JP6.2 (B)
- net at U1.7 (5_IN2): now also JP7.2 (B)
- net at U1.8 (6_OUT1D): now also JP8.2 (B)
- new net: JP43.1 (A), U1.27 (35_TX8)
- new net: JP35.1 (A), U1.36 (14_A0_TX3_SPDIF_OUT)
- new net: JP3.2 (B), U1.3 (1_TX1_CTX2_MISO1)
- new net: JP16.2 (B), U1.17 (25_A11_RX6_SDA2)
- new net: JP44.1 (A), U1.26 (34_RX8)
- new net: JP34.1 (A), U1.37 (15_A1_RX3_SPDIF_IN)
- new net: JP32.1 (A), U1.39 (17_A3_TX4_SDA1)
- new net: JP10.2 (B), U1.10 (8_TX2_IN1)
- new net: JP19.2 (B), U1.20 (28_RX7)
- new net: JP31.1 (A), U1.40 (18_A4_SDA)
- new net: JP15.2 (B), U1.16 (24_A10_TX6_SCL2)
- new net: JP2.2 (B), U1.2 (0_RX1_CRX2_CS1)
- new net: JP20.2 (B), U1.21 (29_TX7)
- new net: JP33.1 (A), U1.38 (16_A2_RX4_SCL1)
- new net: JP30.1 (A), U1.41 (19_A5_SCL)
- new net: JP9.2 (B), U1.9 (7_RX2_OUT1A)
Other:
- moved on the sheet: J16, R20, R21
